File: MSX_4Slot_Expander/MSX_4Slot_Expander.kicad_sch (KiCad schematic)
At the start: 43 parts, among them CN1 MSX_SLOT_CON-msxmakers, CN2 Conn_02x25_Odd_Even_MountingP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, CN3 Conn_02x25_Odd_Even_MountingP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, CN4 Conn_02x25_Odd_Even_MountingP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, CN5 Conn_02x25_Odd_Even_MountingP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, SW1 SW_DIP_x04, U1 74LS30, U2 74LS30, U3 74LS32, U4 74LS240, U5 74LS273, U6 74LS153, U7 74LS139

Commit message: Add files via upload
Added buffers and external +5v supply
Parts:
- removed SW1: SW_DIP_x04, Button_Switch_THT:SW_DIP_SPSTx04_Piano_10.8x11.72mm_W7.62mm_P2.54mm, symbol Switch:SW_DIP_x04
- added C13, C15, C16, C17, C19, C20, C21, C22, C8, C9: 104, Capacitor_THT:C_Disc_D5.0mm_W2.5mm_P5.00mm, symbol Device:C
- added D10, D8, D9: 1N914, Diode_THT:D_DO-35_SOD27_P7.62mm_Horizontal, symbol Diode:1N914
- added JCK1: +5VDC, Connector_BarrelJack:BarrelJack_CUI_PJ-063AH_Horizontal, symbol Connector:Jack-DC
- added JP7: VCC INT, Connector_PinHeader_2.54mm:PinHeader_1x02_P2.54mm_Vertical, symbol Jumper:Jumper_2_Open
- added SW1, SW2, SW3, SW4: SW_Push_DPDT, MSX:SW_PUSH_E-Switch_TL2285_DPDT, symbol Switch:SW_Push_DPDT
- added U10: 74HC245, Package_DIP:DIP-20_W7.62mm_Socket, symbol 74xx:74HC245
- added U11, U12, U13: 74HCT541, Package_DIP:DIP-20_W7.62mm_Socket, symbol 74xx:74HCT541
- added U8: 74HCT32, Package_DIP:DIP-14_W7.62mm_Socket, symbol 74xx:74LS32
- added U9: 74LS08, Package_DIP:DIP-14_W7.62mm_Socket, symbol 74xx:74LS08
- JP1, JP2, JP3, JP4, JP5, JP6: footprint Connector_PinHeader_2.54mm:PinHeader_1x03_P2.54mm_Vertical -> Connector_PinHeader_2.54mm:PinHeader_1x02_P2.54mm_Vertical
- renumbered C9 to C14, C8 to C18
Connections:
- net +5V: now also C10.1, C11.1, C12.1, C13.1, C8.1, C9.1, JP7.1 (A), U10.20 (VCC), U11.20 (VCC), U12.20 (VCC), U13.20 (VCC), U8.14 (VCC), U9.14 (VCC); no longer CN2.45 (Pin_45), CN2.47 (Pin_47), CN3.45 (Pin_45), CN3.47 (Pin_47), CN4.45 (Pin_45), CN4.47 (Pin_47), CN5.45 (Pin_45), CN5.47 (Pin_47)
- net A0: now also U12.2 (A0); no longer CN2.28 (Pin_28), CN3.28 (Pin_28), CN4.28 (Pin_28), CN5.28 (Pin_28), U2.1
- net A1: now also U12.3 (A1); no longer CN2.27 (Pin_27), CN3.27 (Pin_27), CN4.27 (Pin_27), CN5.27 (Pin_27), U2.2
- net A10: now also U13.4 (A2); no longer CN2.20 (Pin_20), CN3.20 (Pin_20), CN4.20 (Pin_20), CN5.20 (Pin_20), U1.1
- net A11: now also U13.5 (A3); no longer CN2.19 (Pin_19), CN3.19 (Pin_19), CN4.19 (Pin_19), CN5.19 (Pin_19), U1.2
- net A12: now also U13.6 (A4); no longer CN2.23 (Pin_23), CN3.23 (Pin_23), CN4.23 (Pin_23), CN5.23 (Pin_23), U1.6
- net A13: now also U13.7 (A5); no longer CN2.26 (Pin_26), CN3.26 (Pin_26), CN4.26 (Pin_26), CN5.26 (Pin_26), U2.12
- net A14: now also U13.8 (A6); no longer CN2.25 (Pin_25), CN3.25 (Pin_25), CN4.25 (Pin_25), CN5.25 (Pin_25), U2.11, U6.14 (S0)
- net A15: now also U13.9 (A7); no longer CN2.18 (Pin_18), CN3.18 (Pin_18), CN4.18 (Pin_18), CN5.18 (Pin_18), U1.12, U6.2 (S1)
- net A2: now also U12.4 (A2); no longer CN2.30 (Pin_30), CN3.30 (Pin_30), CN4.30 (Pin_30), CN5.30 (Pin_30), U2.3
- net A3: now also U12.5 (A3); no longer CN2.29 (Pin_29), CN3.29 (Pin_29), CN4.29 (Pin_29), CN5.29 (Pin_29), U2.4
- net A4: now also U12.6 (A4); no longer CN2.32 (Pin_32), CN3.32 (Pin_32), CN4.32 (Pin_32), CN5.32 (Pin_32), U2.5
- net A5: now also U12.7 (A5); no longer CN2.31 (Pin_31), CN3.31 (Pin_31), CN4.31 (Pin_31), CN5.31 (Pin_31), U2.6
- net A6: now also U12.8 (A6); no longer CN2.22 (Pin_22), CN3.22 (Pin_22), CN4.22 (Pin_22), CN5.22 (Pin_22), U1.3
- net A7: now also U12.9 (A7); no longer CN2.21 (Pin_21), CN3.21 (Pin_21), CN4.21 (Pin_21), CN5.21 (Pin_21), U1.4
- net A8: now also U13.2 (A0); no longer CN2.24 (Pin_24), CN3.24 (Pin_24), CN4.24 (Pin_24), CN5.24 (Pin_24), U1.5
- net A9: now also U13.3 (A1); no longer CN2.17 (Pin_17), CN3.17 (Pin_17), CN4.17 (Pin_17), CN5.17 (Pin_17), U1.11
- net BUSDIR: now also D8.2 (A); no longer CN2.10 (Pin_10), CN3.10 (Pin_10), CN4.10 (Pin_10), CN5.10 (Pin_10)
- net CLK: now also U11.9 (A7); no longer CN2.42 (Pin_42), CN3.42 (Pin_42), CN4.42 (Pin_42), CN5.42 (Pin_42)
- net CS1: now also U9.10, U9.9; no longer CN2.1 (Pin_1), CN3.1 (Pin_1), CN4.1 (Pin_1), CN5.1 (Pin_1)
- net CS12: now also U9.1, U9.2; no longer CN2.3 (Pin_3), CN3.3 (Pin_3), CN4.3 (Pin_3), CN5.3 (Pin_3)
- net CS2: now also U9.4, U9.5; no longer CN2.2 (Pin_2), CN3.2 (Pin_2), CN4.2 (Pin_2), CN5.2 (Pin_2)
- net D0: now also U10.2 (A0); no longer CN2.34 (Pin_34), CN3.34 (Pin_34), CN4.34 (Pin_34), CN5.34 (Pin_34), U4.18 (O0a), U5.3 (D0)
- net D1: now also U10.3 (A1); no longer CN2.33 (Pin_33), CN3.33 (Pin_33), CN4.33 (Pin_33), CN5.33 (Pin_33), U4.16 (O1a), U5.4 (D1)
- net D2: now also U10.4 (A2); no longer CN2.36 (Pin_36), CN3.36 (Pin_36), CN4.36 (Pin_36), CN5.36 (Pin_36), U4.14 (O2a), U5.7 (D2)
- net D3: now also U10.5 (A3); no longer CN2.35 (Pin_35), CN3.35 (Pin_35), CN4.35 (Pin_35), CN5.35 (Pin_35), U4.12 (O3a), U5.8 (D3)
- net D4: now also U10.6 (A4); no longer CN2.38 (Pin_38), CN3.38 (Pin_38), CN4.38 (Pin_38), CN5.38 (Pin_38), U4.9 (O0b), U5.13 (D4)
- net D5: now also U10.7 (A5); no longer CN2.37 (Pin_37), CN3.37 (Pin_37), CN4.37 (Pin_37), CN5.37 (Pin_37), U4.7 (O1b), U5.14 (D5)
- net D6: now also U10.8 (A6); no longer CN2.40 (Pin_40), CN3.40 (Pin_40), CN4.40 (Pin_40), CN5.40 (Pin_40), U4.5 (O2b), U5.17 (D6)
- net D7: now also U10.9 (A7); no longer CN2.39 (Pin_39), CN3.39 (Pin_39), CN4.39 (Pin_39), CN5.39 (Pin_39), U4.3 (O3b), U5.18 (D7)
- net Earth: now also C10.2, C11.2, C12.2, C13.2, C19.2, C20.2, C21.2, C22.2, C8.2, C9.2, JCK1.2, U10.10 (GND), U10.19 (CE), U11.1 (G1), U11.10 (GND), U11.19 (G2), U12.1 (G1), U12.10 (GND), U12.19 (G2), U13.1 (G1), U13.10 (GND), U13.19 (G2), U8.7 (GND), U9.7 (GND)
- net INT: now also D10.2 (A); no longer CN2.8 (Pin_8), CN3.8 (Pin_8), CN4.8 (Pin_8), CN5.8 (Pin_8)
- net IORQ: now also U11.5 (A3); no longer CN2.11 (Pin_11), CN3.11 (Pin_11), CN4.11 (Pin_11), CN5.11 (Pin_11)
- net M1: now also U11.3 (A1); no longer CN2.9 (Pin_9), CN3.9 (Pin_9), CN4.9 (Pin_9), CN5.9 (Pin_9)
- net MERQ: no longer CN2.12 (Pin_12), CN3.12 (Pin_12), CN4.12 (Pin_12), CN5.12 (Pin_12)
- net RD: now also U11.6 (A4), U8.13; no longer CN2.14 (Pin_14), CN3.14 (Pin_14), CN4.14 (Pin_14), CN5.14 (Pin_14), U3.1
- net RESET: now also U11.8 (A6); no longer CN2.15 (Pin_15), CN3.15 (Pin_15), CN4.15 (Pin_15), CN5.15 (Pin_15), U5.1 (~{Mr})
- net RFSH: now also U11.2 (A0); no longer CN2.6 (Pin_6), CN3.6 (Pin_6), CN4.6 (Pin_6), CN5.6 (Pin_6)
- net SLTSL: now also U8.10, U8.12, U8.9; no longer U3.4
- net SLTX0: now also SW1.3 (C); no longer CN3.4 (Pin_4), CN4.4 (Pin_4), CN5.4 (Pin_4), JP1.2 (B), JP5.1 (A)
- net SLTX1: now also CN3.4 (Pin_4), SW2.3 (C); no longer JP2.2 (B), JP5.2 (B)
- net SLTX2: now also CN4.4 (Pin_4), SW3.3 (C); no longer JP3.2 (B), JP6.1 (A)
- net SLTX3: now also CN5.4 (Pin_4), SW4.3 (C); no longer JP4.2 (B), JP6.2 (B)
- net SNDIN: now also C15.2, C16.2, C17.2; no longer C10.2, C11.2, C12.2
- net SW1: no longer CN2.44 (Pin_44), CN3.44 (Pin_44), CN4.44 (Pin_44), CN5.44 (Pin_44)
- net SW2: no longer CN2.46 (Pin_46), CN3.46 (Pin_46), CN4.46 (Pin_46), CN5.46 (Pin_46)
- net WAIT: now also D9.2 (A); no longer CN2.7 (Pin_7), CN3.7 (Pin_7), CN4.7 (Pin_7), CN5.7 (Pin_7)
- net WR: now also U11.7 (A5); no longer CN2.13 (Pin_13), CN3.13 (Pin_13), CN4.13 (Pin_13), CN5.13 (Pin_13), U3.13
- net at CN4.49 (Pin_49): now also C16.1; no longer C11.1
- net at CN5.49 (Pin_49): now also C17.1; no longer C12.1
- net at CN3.49 (Pin_49): now also C15.1; no longer C10.1
- net at JP1.1 (A), U7.12 (O0): now also SW1.2 (B)
- net at JP3.1 (A), U7.10 (O2): now also SW3.2 (B)
- net at JP2.1 (A), U7.11 (O1): now also SW2.2 (B)
- net at JP4.1 (A), U7.9 (O3): now also SW4.2 (B)
- net SLTLS renamed BXSLTLS
- new net: U8.11, U9.13
- new net: JP1.2 (B), JP5.1 (A)
- new net: U10.1 (A->B), U9.11
- new net: D9.1 (K), U8.3
- new net: JP3.2 (B), JP6.1 (A)
- new net: JP4.2 (B), JP6.2 (B)
- new net: JP2.2 (B), JP5.2 (B)
- new net: D10.1 (K), U8.6
- new net +5VS: C19.1, C20.1, C21.1, C22.1, JCK1.1, JP7.2 (B), SW1.5 (B), SW2.5 (B), SW3.5 (B), SW4.5 (B)
- new net +5VS0: CN2.45 (Pin_45), CN2.47 (Pin_47), SW1.6 (C)
- new net +5VS1: CN3.45 (Pin_45), CN3.47 (Pin_47), SW2.6 (C)
- new net +5VS2: CN4.45 (Pin_45), CN4.47 (Pin_47), SW3.6 (C)
- new net +5VS3: CN5.45 (Pin_45), CN5.47 (Pin_47), SW4.6 (C)
- new net BXA0: CN2.28 (Pin_28), CN3.28 (Pin_28), CN4.28 (Pin_28), CN5.28 (Pin_28), U12.18 (Y0), U2.1
- new net BXA1: CN2.27 (Pin_27), CN3.27 (Pin_27), CN4.27 (Pin_27), CN5.27 (Pin_27), U12.17 (Y1), U2.2
- new net BXA10: CN2.20 (Pin_20), CN3.20 (Pin_20), CN4.20 (Pin_20), CN5.20 (Pin_20), U1.1, U13.16 (Y2)
- new net BXA11: CN2.19 (Pin_19), CN3.19 (Pin_19), CN4.19 (Pin_19), CN5.19 (Pin_19), U1.2, U13.15 (Y3)
- new net BXA12: CN2.23 (Pin_23), CN3.23 (Pin_23), CN4.23 (Pin_23), CN5.23 (Pin_23), U1.6, U13.14 (Y4)
- new net BXA13: CN2.26 (Pin_26), CN3.26 (Pin_26), CN4.26 (Pin_26), CN5.26 (Pin_26), U13.13 (Y5), U2.12
- new net BXA14: CN2.25 (Pin_25), CN3.25 (Pin_25), CN4.25 (Pin_25), CN5.25 (Pin_25), U13.12 (Y6), U2.11, U6.14 (S0)
- new net BXA15: CN2.18 (Pin_18), CN3.18 (Pin_18), CN4.18 (Pin_18), CN5.18 (Pin_18), U1.12, U13.11 (Y7), U6.2 (S1)
- new net BXA2: CN2.30 (Pin_30), CN3.30 (Pin_30), CN4.30 (Pin_30), CN5.30 (Pin_30), U12.16 (Y2), U2.3
- new net BXA3: CN2.29 (Pin_29), CN3.29 (Pin_29), CN4.29 (Pin_29), CN5.29 (Pin_29), U12.15 (Y3), U2.4
- new net BXA4: CN2.32 (Pin_32), CN3.32 (Pin_32), CN4.32 (Pin_32), CN5.32 (Pin_32), U12.14 (Y4), U2.5
- new net BXA5: CN2.31 (Pin_31), CN3.31 (Pin_31), CN4.31 (Pin_31), CN5.31 (Pin_31), U12.13 (Y5), U2.6
- new net BXA6: CN2.22 (Pin_22), CN3.22 (Pin_22), CN4.22 (Pin_22), CN5.22 (Pin_22), U1.3, U12.12 (Y6)
- new net BXA7: CN2.21 (Pin_21), CN3.21 (Pin_21), CN4.21 (Pin_21), CN5.21 (Pin_21), U1.4, U12.11 (Y7)
- new net BXA8: CN2.24 (Pin_24), CN3.24 (Pin_24), CN4.24 (Pin_24), CN5.24 (Pin_24), U1.5, U13.18 (Y0)
- new net BXA9: CN2.17 (Pin_17), CN3.17 (Pin_17), CN4.17 (Pin_17), CN5.17 (Pin_17), U1.11, U13.17 (Y1)
- new net BXCLK: CN2.42 (Pin_42), CN3.42 (Pin_42), CN4.42 (Pin_42), CN5.42 (Pin_42), U11.11 (Y7)
- new net BXCS1: CN2.1 (Pin_1), CN3.1 (Pin_1), CN4.1 (Pin_1), CN5.1 (Pin_1), U9.8
- new net BXCS12: CN2.3 (Pin_3), CN3.3 (Pin_3), CN4.3 (Pin_3), CN5.3 (Pin_3), U9.3
- new net BXCS2: CN2.2 (Pin_2), CN3.2 (Pin_2), CN4.2 (Pin_2), CN5.2 (Pin_2), U9.6
- new net BXD0: CN2.34 (Pin_34), CN3.34 (Pin_34), CN4.34 (Pin_34), CN5.34 (Pin_34), U10.18 (B0), U4.18 (O0a), U5.3 (D0)
- new net BXD1: CN2.33 (Pin_33), CN3.33 (Pin_33), CN4.33 (Pin_33), CN5.33 (Pin_33), U10.17 (B1), U4.16 (O1a), U5.4 (D1)
- new net BXD2: CN2.36 (Pin_36), CN3.36 (Pin_36), CN4.36 (Pin_36), CN5.36 (Pin_36), U10.16 (B2), U4.14 (O2a), U5.7 (D2)
- new net BXD3: CN2.35 (Pin_35), CN3.35 (Pin_35), CN4.35 (Pin_35), CN5.35 (Pin_35), U10.15 (B3), U4.12 (O3a), U5.8 (D3)
- new net BXD4: CN2.38 (Pin_38), CN3.38 (Pin_38), CN4.38 (Pin_38), CN5.38 (Pin_38), U10.14 (B4), U4.9 (O0b), U5.13 (D4)
- new net BXD5: CN2.37 (Pin_37), CN3.37 (Pin_37), CN4.37 (Pin_37), CN5.37 (Pin_37), U10.13 (B5), U4.7 (O1b), U5.14 (D5)
- new net BXD6: CN2.40 (Pin_40), CN3.40 (Pin_40), CN4.40 (Pin_40), CN5.40 (Pin_40), U10.12 (B6), U4.5 (O2b), U5.17 (D6)
- new net BXD7: CN2.39 (Pin_39), CN3.39 (Pin_39), CN4.39 (Pin_39), CN5.39 (Pin_39), U10.11 (B7), U4.3 (O3b), U5.18 (D7)
- new net BXDIR: CN2.10 (Pin_10), CN3.10 (Pin_10), CN4.10 (Pin_10), CN5.10 (Pin_10), D8.1 (K), U9.12
- new net BXINT: CN2.8 (Pin_8), CN3.8 (Pin_8), CN4.8 (Pin_8), CN5.8 (Pin_8), U8.4, U8.5
- new net BXIORQ: CN2.11 (Pin_11), CN3.11 (Pin_11), CN4.11 (Pin_11), CN5.11 (Pin_11), U11.15 (Y3)
- new net BXM1: CN2.9 (Pin_9), CN3.9 (Pin_9), CN4.9 (Pin_9), CN5.9 (Pin_9), U11.17 (Y1)
- new net BXMERQ: CN2.12 (Pin_12), CN3.12 (Pin_12), CN4.12 (Pin_12), CN5.12 (Pin_12)
- new net BXMREQ: U11.16 (Y2)
- new net BXRD: CN2.14 (Pin_14), CN3.14 (Pin_14), CN4.14 (Pin_14), CN5.14 (Pin_14), U11.14 (Y4), U3.1
- new net BXRESET: CN2.15 (Pin_15), CN3.15 (Pin_15), CN4.15 (Pin_15), CN5.15 (Pin_15), U11.12 (Y6), U5.1 (~{Mr})
- new net BXRFSH: CN2.6 (Pin_6), CN3.6 (Pin_6), CN4.6 (Pin_6), CN5.6 (Pin_6), U11.18 (Y0)
- new net BXSLTSL: U3.4, U8.8
- new net BXWAIT: CN2.7 (Pin_7), CN3.7 (Pin_7), CN4.7 (Pin_7), CN5.7 (Pin_7), U8.1, U8.2
- new net BXWR: CN2.13 (Pin_13), CN3.13 (Pin_13), CN4.13 (Pin_13), CN5.13 (Pin_13), U11.13 (Y5), U3.13
- new net MREQ: U11.4 (A2)
- new net SW10: CN2.44 (Pin_44)
- new net SW11: CN3.44 (Pin_44)
- new net SW12: CN4.44 (Pin_44)
- new net SW13: CN5.44 (Pin_44)
- new net SW20: CN2.46 (Pin_46)
- new net SW21: CN3.46 (Pin_46)
- new net SW22: CN4.46 (Pin_46)
- new net SW23: CN5.46 (Pin_46)
Other:
- note added: "Buffer"
- company: (none) -> Luis Vina
- moved on the sheet: C1, C14, C18, C2, C3, C4, C5, C6, C7, CN2, D1, D2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

Commit message: Add files via upload
Parts:
- removed C19, C20, C21, C22: 104, Capacitor_THT:C_Disc_D5.0mm_W2.5mm_P5.00mm, symbol Device:C
- removed D1, D2, D3: 1N914, Diode_THT:D_DO-35_SOD27_P7.62mm_Horizontal, symbol Diode:1N914
- removed JP7: VCC INT, Connector_PinHeader_2.54mm:PinHeader_1x02_P2.54mm_Vertical, symbol Jumper:Jumper_2_Open
- removed R1: 1K, Resistor_THT:R_Axial_DIN0207_L6.3mm_D2.5mm_P7.62mm_Horizontal, symbol Device:R
- removed SW1, SW2, SW3, SW4: SW_Push_DPDT, MSX:SW_PUSH_E-Switch_TL2285_DPDT, symbol Switch:SW_Push_DPDT
- added C14, C15, C16: 104, Capacitor_THT:C_Disc_D5.0mm_W2.5mm_P5.00mm, symbol Device:C
- added C22: 100uF, Capacitor_THT:CP_Radial_D6.3mm_P2.50mm, symbol Device:C_Polarized
- added PS1: IH0512D, Converter_DCDC:Converter_DCDC_XP_POWER-IHxxxxD_THT, symbol Converter_DCDC:IH0512D
- added SW1, SW2, SW3, SW5: SW_Push_4PDT, MSX:Push Switch 4P2T SPUJ193700, symbol msx_slot_con-msxmakers:SW_Push_4PDT
- added U11: 74LS11, Package_DIP:DIP-14_W7.62mm_Socket, symbol 74xx:74LS11
- added U12: 74LS08, Package_DIP:DIP-14_W7.62mm_Socket, symbol 74xx:74LS08
- added U13: 74LS32, Package_DIP:DIP-14_W7.62mm_Socket, symbol 74xx:74LS32
- added U17, U18, U19: AQH0223, Package_DIP:DIP-8-N7_W7.62mm, symbol Relay_SolidState:AQH0223
- renumbered C14 to C17, C15 to C18, C16 to C19, C17 to C20, C18 to C21, U10 to U1, U3 to U10, U5 to U14, U4 to U15, U6 to U16, U11 to U2, U12 to U3, U13 to U4, U9 to U5, U8 to U6, U1 to U7, U2 to U8, U7 to U9
Connections:
- net +12V: no longer CN2.48 (Pin_48), CN3.48 (Pin_48), CN4.48 (Pin_48), CN5.48 (Pin_48)
- net +5V: now also C22.1, U17.6; no longer C10.1, C11.1, C12.1, C13.1, C21.1, C7.1, C8.1, C9.1, R2.1, R3.1, R4.1, R5.1, U10.14 (VCC), U14.20 (VCC), U15.20 (VCC), U16.16 (VCC), U7.14 (VCC), U8.14 (VCC), U9.16 (VCC)
- net +5VS: now also C10.1, C11.1, C12.1, C13.1, C21.1, C7.1, C8.1, C9.1, R2.1, R3.1, R4.1, R5.1, U10.14 (VCC), U14.20 (VCC), U15.20 (VCC), U16.16 (VCC), U7.14 (VCC), U8.14 (VCC), U9.16 (VCC), C14.1, C15.1, C16.1, SW1.5 (B), SW2.5 (B), SW3.5 (B), SW5.5 (B), U11.14 (VCC), U12.14 (VCC), U13.14 (VCC), U17.8; no longer JCK1.1
- net +5VS0: now also SW5.6 (C)
- net +5VS1: now also SW1.6 (C)
- net +5VS2: now also SW2.6 (C)
- net +5VS3: now also SW3.6 (C)
- net -12V: now also U19.6; no longer CN2.50 (Pin_50), CN3.50 (Pin_50), CN4.50 (Pin_50), CN5.50 (Pin_50)
- net BXDIR: now also U11.12; no longer CN2.10 (Pin_10), CN3.10 (Pin_10), CN4.10 (Pin_10), CN5.10 (Pin_10)
- net BXRD: now also U13.2
- net BXSLTSL: now also U13.1
- net Earth: now also C14.2, C15.2, C16.2, C22.2, PS1.1 (-Vin), PS1.6 (0V), U17.1, U17.3, U17.4, U18.1, U18.3, U18.4, U19.1, U19.3, U19.4
- net SLTX0: now also SW5.3 (C)
- net SLTX1: now also SW1.1 (A)
- net SLTX2: now also SW2.1 (A)
- net SLTX3: now also SW3.1 (A)
- net at JP4.1 (A), U9.9 (O3): now also SW3.2 (B)
- net at JP3.1 (A), U9.10 (O2): now also SW2.2 (B)
- net at U10.9: now also U11.6
- net at JP1.1 (A), U9.12 (O0): now also SW5.2 (B)
- net at JP2.1 (A), U9.11 (O1): now also SW1.2 (B)
- net at U9.5 (O1): now also U11.3
- net at U9.6 (O2): now also U11.4
- net at U9.7 (O3): now also U11.5
- new net: JCK1.1, PS1.3 (+Vin), U17.2, U17.5, U18.2, U19.2
- new net: PS1.5 (+Vout), U18.5
- new net: U11.1, U13.3
- new net: U11.13, U12.3
- new net: U11.2, U12.6
- new net: PS1.4 (-Vout), U19.5
- new net +12VS: SW1.8 (B), SW2.8 (B), SW3.8 (B), SW5.8 (B), U18.8
- new net +12VS0: CN2.48 (Pin_48), SW5.9 (C)
- new net +12VS1: CN3.48 (Pin_48), SW1.9 (C)
- new net +12VS2: CN4.48 (Pin_48), SW2.9 (C)
- new net +12VS3: CN5.48 (Pin_48), SW3.9 (C)
- new net +12v: U18.6
- new net -12VS: SW1.11 (B), SW2.11 (B), SW3.11 (B), SW5.11 (B), U19.8
- new net -12VS0: CN2.50 (Pin_50), SW5.12 (C)
- new net -12VS1: CN3.50 (Pin_50), SW1.12 (C)
- new net -12VS2: CN4.50 (Pin_50), SW2.12 (C)
- new net -12VS3: CN5.50 (Pin_50), SW3.12 (C)
- new net BXDIR0: CN2.10 (Pin_10), U12.2
- new net BXDIR1: CN3.10 (Pin_10), U12.1
- new net BXDIR2: CN4.10 (Pin_10), U12.5
- new net BXDIR3: CN5.10 (Pin_10), U12.4
Other:
- note removed: "OBS: Project based on CIEL A13713 de Ademir Carchano"
- moved on the sheet: C1, C10, C11, C12, C13, C2, C21, C3, C4, C5, C6, C7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
